Commit message: feat: Add bartender robot model with RViz configuration and Gazebo integration

File: urdf/bartender_robot.xacro (robot description, xacro)
@@ -1,7 +1,7 @@
 <?xml version="1.0" ?>
-<robot name="test_assembly3" xmlns:xacro="http://www.ros.org/wiki/xacro">
-<xacro:include filename="$(find test_assembly3_description)/urdf/materials.xacro" />
-<xacro:include filename="$(find test_assembly3_description)/urdf/test_assembly3.trans" />
-<xacro:include filename="$(find test_assembly3_description)/urdf/test_assembly3.gazebo" />
+<robot name="bartender_robot" xmlns:xacro="http://www.ros.org/wiki/xacro">
+<xacro:include filename="$(find bartender_robot)/urdf/materials.xacro" />
+<xacro:include filename="$(find bartender_robot)/urdf/bartender_robot.trans" />
+<xacro:include filename="$(find bartender_robot)/urdf/bartender_robot.gazebo" />
 <link name="base_link">
   <inertial>
@@ -13,5 +13,5 @@
     <origin xyz="0 0 0" rpy="0 0 0"/>
     <geometry>
-      <mesh filename="package://test_assembly3_description/meshes/base_link.stl" scale="0.001 0.001 0.001"/>
+  <mesh filename="package://bartender_robot/meshes/base_link.stl" scale="0.001 0.001 0.001"/>
     </geometry>
     <material name="silver"/>
@@ -20,5 +20,5 @@
     <origin xyz="0 0 0" rpy="0 0 0"/>
     <geometry>
-      <mesh filename="package://test_assembly3_description/meshes/base_link.stl" scale="0.001 0.001 0.001"/>
+      <mesh filename="package://bartender_robot/meshes/base_link.stl" scale="0.001 0.001 0.001"/>
     </geometry>
   </collision>
@@ -33,5 +33,5 @@
     <origin xyz="0.0 0.0 -0.015" rpy="0 0 0"/>
     <geometry>
-      <mesh filename="package://test_assembly3_description/meshes/motor_base_1.stl" scale="0.001 0.001 0.001"/>
+  <mesh filename="package://bartender_robot/meshes/motor_base_1.stl" scale="0.001 0.001 0.001"/>
     </geometry>
     <material name="silver"/>
@@ -40,5 +40,5 @@
     <origin xyz="0.0 0.0 -0.015" rpy="0 0 0"/>
     <geometry>
-      <mesh filename="package://test_assembly3_description/meshes/motor_base_1.stl" scale="0.001 0.001 0.001"/>
+      <mesh filename="package://bartender_robot/meshes/motor_base_1.stl" scale="0.001 0.001 0.001"/>
     </geometry>
   </collision>
@@ -53,5 +53,5 @@
     <origin xyz="0.0 0.0 -0.041" rpy="0 0 0"/>
     <geometry>
-      <mesh filename="package://test_assembly3_description/meshes/base_upperplate_1.stl" scale="0.001 0.001 0.001"/>
+  <mesh filename="package://bartender_robot/meshes/base_upperplate_1.stl" scale="0.001 0.001 0.001"/>
     </geometry>
     <material name="silver"/>
@@ -60,5 +60,5 @@
     <origin xyz="0.0 0.0 -0.041" rpy="0 0 0"/>
     <geometry>
-      <mesh filename="package://test_assembly3_description/meshes/base_upperplate_1.stl" scale="0.001 0.001 0.001"/>
+      <mesh filename="package://bartender_robot/meshes/base_upperplate_1.stl" scale="0.001 0.001 0.001"/>
     </geometry>
   </collision>
@@ -73,5 +73,5 @@
     <origin xyz="0.0 0.0 -0.0475" rpy="0 0 0"/>
     <geometry>
-      <mesh filename="package://test_assembly3_description/meshes/motor_horn_base_1.stl" scale="0.001 0.001 0.001"/>
+  <mesh filename="package://bartender_robot/meshes/motor_horn_base_1.stl" scale="0.001 0.001 0.001"/>
     </geometry>
     <material name="silver"/>
@@ -80,5 +80,5 @@
     <origin xyz="0.0 0.0 -0.0475" rpy="0 0 0"/>
     <geometry>
-      <mesh filename="package://test_assembly3_description/meshes/motor_horn_base_1.stl" scale="0.001 0.001 0.001"/>
+      <mesh filename="package://bartender_robot/meshes/motor_horn_base_1.stl" scale="0.001 0.001 0.001"/>
     </geometry>
   </collision>
@@ -93,5 +93,5 @@
     <origin xyz="0.0 0.0 -0.051" rpy="0 0 0"/>
     <geometry>
-      <mesh filename="package://test_assembly3_description/meshes/link1_1.stl" scale="0.001 0.001 0.001"/>
+      <mesh filename="package://bartender_robot/meshes/link1_1.stl" scale="0.001 0.001 0.001"/>
     </geometry>
     <material name="silver"/>
@@ -100,5 +100,5 @@
     <origin xyz="0.0 0.0 -0.051" rpy="0 0 0"/>
     <geometry>
-      <mesh filename="package://test_assembly3_description/meshes/link1_1.stl" scale="0.001 0.001 0.001"/>
+      <mesh filename="package://bartender_robot/meshes/link1_1.stl" scale="0.001 0.001 0.001"/>
     </geometry>
   </collision>
@@ -113,5 +113,5 @@
     <origin xyz="0.023374 0.016412 -0.15725" rpy="0 0 0"/>
     <geometry>
-      <mesh filename="package://test_assembly3_description/meshes/motor_fix_link1_1.stl" scale="0.001 0.001 0.001"/>
+      <mesh filename="package://bartender_robot/meshes/motor_fix_link1_1.stl" scale="0.001 0.001 0.001"/>
     </geometry>
     <material name="silver"/>
@@ -120,5 +120,5 @@
     <origin xyz="0.023374 0.016412 -0.15725" rpy="0 0 0"/>
     <geometry>
-      <mesh filename="package://test_assembly3_description/meshes/motor_fix_link1_1.stl" scale="0.001 0.001 0.001"/>
+      <mesh filename="package://bartender_robot/meshes/motor_fix_link1_1.stl" scale="0.001 0.001 0.001"/>
     </geometry>
   </collision>
@@ -133,5 +133,5 @@
     <origin xyz="0.023584 0.01518 -0.149" rpy="0 0 0"/>
     <geometry>
-      <mesh filename="package://test_assembly3_description/meshes/motor_link1_1.stl" scale="0.001 0.001 0.001"/>
+      <mesh filename="package://bartender_robot/meshes/motor_link1_1.stl" scale="0.001 0.001 0.001"/>
     </geometry>
     <material name="silver"/>
@@ -140,5 +140,5 @@
     <origin xyz="0.023584 0.01518 -0.149" rpy="0 0 0"/>
     <geometry>
-      <mesh filename="package://test_assembly3_description/meshes/motor_link1_1.stl" scale="0.001 0.001 0.001"/>
+      <mesh filename="package://bartender_robot/meshes/motor_link1_1.stl" scale="0.001 0.001 0.001"/>
     </geometry>
   </collision>
@@ -153,5 +153,5 @@
     <origin xyz="0.024152 0.004118 -0.141" rpy="0 0 0"/>
     <geometry>
-      <mesh filename="package://test_assembly3_description/meshes/motor_horn_link1_1.stl" scale="0.001 0.001 0.001"/>
+      <mesh filename="package://bartender_robot/meshes/motor_horn_link1_1.stl" scale="0.001 0.001 0.001"/>
     </geometry>
     <material name="silver"/>
@@ -160,5 +160,5 @@
     <origin xyz="0.024152 0.004118 -0.141" rpy="0 0 0"/>
     <geometry>
-      <mesh filename="package://test_assembly3_description/meshes/motor_horn_link1_1.stl" scale="0.001 0.001 0.001"/>
+      <mesh filename="package://bartender_robot/meshes/motor_horn_link1_1.stl" scale="0.001 0.001 0.001"/>
     </geometry>
   </collision>
@@ -173,5 +173,5 @@
     <origin xyz="0.020701 0.003529 -0.141" rpy="0 0 0"/>
     <geometry>
-      <mesh filename="package://test_assembly3_description/meshes/link2_1.stl" scale="0.001 0.001 0.001"/>
+      <mesh filename="package://bartender_robot/meshes/link2_1.stl" scale="0.001 0.001 0.001"/>
     </geometry>
     <material name="silver"/>
@@ -180,5 +180,5 @@
     <origin xyz="0.020701 0.003529 -0.141" rpy="0 0 0"/>
     <geometry>
-      <mesh filename="package://test_assembly3_description/meshes/link2_1.stl" scale="0.001 0.001 0.001"/>
+      <mesh filename="package://bartender_robot/meshes/link2_1.stl" scale="0.001 0.001 0.001"/>
     </geometry>
   </collision>
@@ -193,5 +193,5 @@
     <origin xyz="0.015263 -0.018122 -0.147219" rpy="0 0 0"/>
     <geometry>
-      <mesh filename="package://test_assembly3_description/meshes/motor_link2_1.stl" scale="0.001 0.001 0.001"/>
+      <mesh filename="package://bartender_robot/meshes/motor_link2_1.stl" scale="0.001 0.001 0.001"/>
     </geometry>
     <material name="silver"/>
@@ -200,5 +200,5 @@
     <origin xyz="0.015263 -0.018122 -0.147219" rpy="0 0 0"/>
     <geometry>
-      <mesh filename="package://test_assembly3_description/meshes/motor_link2_1.stl" scale="0.001 0.001 0.001"/>
+      <mesh filename="package://bartender_robot/meshes/motor_link2_1.stl" scale="0.001 0.001 0.001"/>
     </geometry>
   </collision>
@@ -213,5 +213,5 @@
     <origin xyz="0.004083 -0.017997 -0.139365" rpy="0 0 0"/>
     <geometry>
-      <mesh filename="package://test_assembly3_description/meshes/motor_horn_link2_1.stl" scale="0.001 0.001 0.001"/>
+      <mesh filename="package://bartender_robot/meshes/motor_horn_link2_1.stl" scale="0.001 0.001 0.001"/>
     </geometry>
     <material name="silver"/>
@@ -220,5 +220,5 @@
     <origin xyz="0.004083 -0.017997 -0.139365" rpy="0 0 0"/>
     <geometry>
-      <mesh filename="package://test_assembly3_description/meshes/motor_horn_link2_1.stl" scale="0.001 0.001 0.001"/>
+      <mesh filename="package://bartender_robot/meshes/motor_horn_link2_1.stl" scale="0.001 0.001 0.001"/>
     </geometry>
   </collision>
@@ -233,5 +233,5 @@
     <origin xyz="0.003497 -0.014561 -0.139674" rpy="0 0 0"/>
     <geometry>
-      <mesh filename="package://test_assembly3_description/meshes/link3_1.stl" scale="0.001 0.001 0.001"/>
+      <mesh filename="package://bartender_robot/meshes/link3_1.stl" scale="0.001 0.001 0.001"/>
     </geometry>
     <material name="silver"/>
@@ -240,5 +240,5 @@
     <origin xyz="0.003497 -0.014561 -0.139674" rpy="0 0 0"/>
     <geometry>
-      <mesh filename="package://test_assembly3_description/meshes/link3_1.stl" scale="0.001 0.001 0.001"/>
+      <mesh filename="package://bartender_robot/meshes/link3_1.stl" scale="0.001 0.001 0.001"/>
     </geometry>
   </collision>
@@ -253,5 +253,5 @@
     <origin xyz="-0.023288 0.142546 -0.153815" rpy="0 0 0"/>
     <geometry>
-      <mesh filename="package://test_assembly3_description/meshes/motor_fix_link3_1.stl" scale="0.001 0.001 0.001"/>
+      <mesh filename="package://bartender_robot/meshes/motor_fix_link3_1.stl" scale="0.001 0.001 0.001"/>
     </geometry>
     <material name="silver"/>
@@ -260,5 +260,5 @@
     <origin xyz="-0.023288 0.142546 -0.153815" rpy="0 0 0"/>
     <geometry>
-      <mesh filename="package://test_assembly3_description/meshes/motor_fix_link3_1.stl" scale="0.001 0.001 0.001"/>
+      <mesh filename="package://bartender_robot/meshes/motor_fix_link3_1.stl" scale="0.001 0.001 0.001"/>
     </geometry>
   </collision>
@@ -273,5 +273,5 @@
     <origin xyz="-0.015046 0.148117 -0.164112" rpy="0 0 0"/>
     <geometry>
-      <mesh filename="package://test_assembly3_description/meshes/motor_link3_1.stl" scale="0.001 0.001 0.001"/>
+      <mesh filename="package://bartender_robot/meshes/motor_link3_1.stl" scale="0.001 0.001 0.001"/>
     </geometry>
     <material name="silver"/>
@@ -280,5 +280,5 @@
     <origin xyz="-0.015046 0.148117 -0.164112" rpy="0 0 0"/>
     <geometry>
-      <mesh filename="package://test_assembly3_description/meshes/motor_link3_1.stl" scale="0.001 0.001 0.001"/>
+      <mesh filename="package://bartender_robot/meshes/motor_link3_1.stl" scale="0.001 0.001 0.001"/>
     </geometry>
   </collision>
@@ -293,5 +293,5 @@
     <origin xyz="-0.036587 0.15797 -0.175077" rpy="0 0 0"/>
     <geometry>
-      <mesh filename="package://test_assembly3_description/meshes/motor_horn_link3_1.stl" scale="0.001 0.001 0.001"/>
+      <mesh filename="package://bartender_robot/meshes/motor_horn_link3_1.stl" scale="0.001 0.001 0.001"/>
     </geometry>
     <material name="silver"/>
@@ -300,5 +300,5 @@
     <origin xyz="-0.036587 0.15797 -0.175077" rpy="0 0 0"/>
     <geometry>
-      <mesh filename="package://test_assembly3_description/meshes/motor_horn_link3_1.stl" scale="0.001 0.001 0.001"/>
+      <mesh filename="package://bartender_robot/meshes/motor_horn_link3_1.stl" scale="0.001 0.001 0.001"/>
     </geometry>
   </collision>
@@ -313,5 +313,5 @@
     <origin xyz="-0.03989 0.15732 -0.176033" rpy="0 0 0"/>
     <geometry>
-      <mesh filename="package://test_assembly3_description/meshes/link4_1.stl" scale="0.001 0.001 0.001"/>
+      <mesh filename="package://bartender_robot/meshes/link4_1.stl" scale="0.001 0.001 0.001"/>
     </geometry>
     <material name="silver"/>
@@ -320,5 +320,5 @@
     <origin xyz="-0.03989 0.15732 -0.176033" rpy="0 0 0"/>
     <geometry>
-      <mesh filename="package://test_assembly3_description/meshes/link4_1.stl" scale="0.001 0.001 0.001"/>
+      <mesh filename="package://bartender_robot/meshes/link4_1.stl" scale="0.001 0.001 0.001"/>
     </geometry>
   </collision>
@@ -333,5 +333,5 @@
     <origin xyz="-0.060395 0.332013 -0.17623" rpy="0 0 0"/>
     <geometry>
-      <mesh filename="package://test_assembly3_description/meshes/motor_link4_1.stl" scale="0.001 0.001 0.001"/>
+      <mesh filename="package://bartender_robot/meshes/motor_link4_1.stl" scale="0.001 0.001 0.001"/>
     </geometry>
     <material name="silver"/>
@@ -340,5 +340,5 @@
     <origin xyz="-0.060395 0.332013 -0.17623" rpy="0 0 0"/>
     <geometry>
-      <mesh filename="package://test_assembly3_description/meshes/motor_link4_1.stl" scale="0.001 0.001 0.001"/>
+      <mesh filename="package://bartender_robot/meshes/motor_link4_1.stl" scale="0.001 0.001 0.001"/>
     </geometry>
   </collision>
@@ -353,5 +353,5 @@
     <origin xyz="-0.056813 0.327062 -0.163282" rpy="0 0 0"/>
     <geometry>
-      <mesh filename="package://test_assembly3_description/meshes/motor_fix_link4_1.stl" scale="0.001 0.001 0.001"/>
+      <mesh filename="package://bartender_robot/meshes/motor_fix_link4_1.stl" scale="0.001 0.001 0.001"/>
     </geometry>
     <material name="silver"/>
@@ -360,5 +360,5 @@
     <origin xyz="-0.056813 0.327062 -0.163282" rpy="0 0 0"/>
     <geometry>
-      <mesh filename="package://test_assembly3_description/meshes/motor_fix_link4_1.stl" scale="0.001 0.001 0.001"/>
+      <mesh filename="package://bartender_robot/meshes/motor_fix_link4_1.stl" scale="0.001 0.001 0.001"/>
     </geometry>
   </collision>
@@ -373,5 +373,5 @@
     <origin xyz="-0.071249 0.344576 -0.182036" rpy="0 0 0"/>
     <geometry>
-      <mesh filename="package://test_assembly3_description/meshes/motor_horn_link4_1.stl" scale="0.001 0.001 0.001"/>
+      <mesh filename="package://bartender_robot/meshes/motor_horn_link4_1.stl" scale="0.001 0.001 0.001"/>
     </geometry>
     <material name="silver"/>
@@ -380,5 +380,5 @@
     <origin xyz="-0.071249 0.344576 -0.182036" rpy="0 0 0"/>
     <geometry>
-      <mesh filename="package://test_assembly3_description/meshes/motor_horn_link4_1.stl" scale="0.001 0.001 0.001"/>
+      <mesh filename="package://bartender_robot/meshes/motor_horn_link4_1.stl" scale="0.001 0.001 0.001"/>
     </geometry>
   </collision>

File: urdf/materials.xacro (robot description, xacro)
@@ -1,4 +1,4 @@
 <?xml version="1.0" ?>
-<robot name="test_assembly3" xmlns:xacro="http://www.ros.org/wiki/xacro" >
+<robot name="bartender_robot" xmlns:xacro="http://www.ros.org/wiki/xacro" >
 <material name="silver">
   <color rgba="0.700 0.700 0.700 1.000"/>
