Commit message: fix: update urdf

File: urdf/bartender_robot.xacro (robot description, xacro)
@@ -2,14 +2,16 @@
 <robot name="bartender_robot" xmlns:xacro="http://www.ros.org/wiki/xacro">
 <xacro:include filename="$(find bartender_robot)/urdf/materials.xacro" />
+<xacro:include filename="$(find bartender_robot)/urdf/bartender_robot.trans.xacro" />
+<xacro:include filename="$(find bartender_robot)/urdf/bartender_robot.gazebo" />
 <link name="base_link">
   <inertial>
-    <origin xyz="-0.00040810804018468253 -3.552713678800501e-17 0.016706580181223032" rpy="0 0 0"/>
-    <mass value="6.935188631739772"/>
-    <inertia ixx="0.028142" iyy="0.028238" izz="0.054243" ixy="-0.0" iyz="-0.0" ixz="2.5e-05"/>
+    <origin xyz="-0.04417987256972955 0.006609684065759414 0.01837618890169653" rpy="0 0 0"/>
+    <mass value="1.8079552496262556"/>
+    <inertia ixx="0.006993" iyy="0.007027" izz="0.013194" ixy="0.0" iyz="-0.0" ixz="3e-06"/>
   </inertial>
   <visual>
     <origin xyz="0 0 0" rpy="0 0 0"/>
     <geometry>
-  <mesh filename="package://bartender_robot/meshes/base_link.stl" scale="0.001 0.001 0.001"/>
+      <mesh filename="$(find bartender_robot)/meshes/base_link.stl" scale="0.001 0.001 0.001"/>
     </geometry>
     <material name="silver"/>
@@ -18,462 +20,1119 @@
     <origin xyz="0 0 0" rpy="0 0 0"/>
     <geometry>
-      <mesh filename="package://bartender_robot/meshes/base_link.stl" scale="0.001 0.001 0.001"/>
-    </geometry>
-  </collision>
-</link>
-<link name="motor_base_1">
-  <inertial>
-    <origin xyz="-0.011944616237443872 -1.1102230246251566e-17 0.016403799171755752" rpy="0 0 0"/>
-    <mass value="0.343534365338019"/>
-    <inertia ixx="5.5e-05" iyy="9.2e-05" izz="8.2e-05" ixy="-0.0" iyz="0.0" ixz="2e-06"/>
-  </inertial>
-  <visual>
-    <origin xyz="0.0 0.0 -0.015" rpy="0 0 0"/>
-    <geometry>
-  <mesh filename="package://bartender_robot/meshes/motor_base_1.stl" scale="0.001 0.001 0.001"/>
-    </geometry>
-    <material name="silver"/>
-  </visual>
-  <collision>
-    <origin xyz="0.0 0.0 -0.015" rpy="0 0 0"/>
-    <geometry>
-      <mesh filename="package://bartender_robot/meshes/motor_base_1.stl" scale="0.001 0.001 0.001"/>
-    </geometry>
-  </collision>
-</link>
-<link name="base_upperplate_1">
-  <inertial>
-    <origin xyz="-1.6172448750803435e-16 -3.676205142934621e-17 0.004999999999999949" rpy="0 0 0"/>
-    <mass value="1.9420933085410403"/>
-    <inertia ixx="0.007942" iyy="0.007942" izz="0.015852" ixy="-0.0" iyz="0.0" ixz="0.0"/>
-  </inertial>
-  <visual>
-    <origin xyz="0.0 0.0 -0.041" rpy="0 0 0"/>
-    <geometry>
-  <mesh filename="package://bartender_robot/meshes/base_upperplate_1.stl" scale="0.001 0.001 0.001"/>
-    </geometry>
-    <material name="silver"/>
-  </visual>
-  <collision>
-    <origin xyz="0.0 0.0 -0.041" rpy="0 0 0"/>
-    <geometry>
-      <mesh filename="package://bartender_robot/meshes/base_upperplate_1.stl" scale="0.001 0.001 0.001"/>
-    </geometry>
-  </collision>
-</link>
-<link name="motor_horn_base_1">
-  <inertial>
-    <origin xyz="3.138091383686708e-14 5.3428299048114016e-15 0.0019561696415957355" rpy="0 0 0"/>
+      <mesh filename="$(find bartender_robot)/meshes/base_link.stl" scale="0.001 0.001 0.001"/>
+    </geometry>
+  </collision>
+</link>
+<link name="XL_430_base_1">
+  <inertial>
+    <origin xyz="-0.011917916373983276 -1.4051646660215994e-07 0.016402708590339682" rpy="0 0 0"/>
+    <mass value="0.34309933643690577"/>
+    <inertia ixx="5.5e-05" iyy="9.2e-05" izz="8.2e-05" ixy="0.0" iyz="-0.0" ixz="2e-06"/>
+  </inertial>
+  <visual>
+    <origin xyz="0.043637 -0.006593 -0.009671" rpy="0 0 0"/>
+    <geometry>
+      <mesh filename="$(find bartender_robot)/meshes/XL_430_base_1.stl" scale="0.001 0.001 0.001"/>
+    </geometry>
+    <material name="silver"/>
+  </visual>
+  <collision>
+    <origin xyz="0.043637 -0.006593 -0.009671" rpy="0 0 0"/>
+    <geometry>
+      <mesh filename="$(find bartender_robot)/meshes/XL_430_base_1.stl" scale="0.001 0.001 0.001"/>
+    </geometry>
+  </collision>
+</link>
+<link name="horn_base_1">
+  <inertial>
+    <origin xyz="-3.140555788552768e-07 -1.4051646675915241e-07 0.0019558350062390192" rpy="0 0 0"/>
+    <mass value="0.009818206481012393"/>
+    <inertia ixx="0.0" iyy="0.0" izz="0.0" ixy="0.0" iyz="0.0" ixz="0.0"/>
+  </inertial>
+  <visual>
+    <origin xyz="0.043637 -0.006593 -0.042171" rpy="0 0 0"/>
+    <geometry>
+      <mesh filename="$(find bartender_robot)/meshes/horn_base_1.stl" scale="0.001 0.001 0.001"/>
+    </geometry>
+    <material name="silver"/>
+  </visual>
+  <collision>
+    <origin xyz="0.043637 -0.006593 -0.042171" rpy="0 0 0"/>
+    <geometry>
+      <mesh filename="$(find bartender_robot)/meshes/horn_base_1.stl" scale="0.001 0.001 0.001"/>
+    </geometry>
+  </collision>
+</link>
+<link name="shoulder_base_1">
+  <inertial>
+    <origin xyz="-3.14055541496272e-07 -1.4051646674961144e-07 0.00501347381325503" rpy="0 0 0"/>
+    <mass value="0.38517204561220847"/>
+    <inertia ixx="0.000968" iyy="0.000958" izz="0.00192" ixy="0.0" iyz="0.0" ixz="-0.0"/>
+  </inertial>
+  <visual>
+    <origin xyz="0.043637 -0.006593 -0.045671" rpy="0 0 0"/>
+    <geometry>
+      <mesh filename="$(find bartender_robot)/meshes/shoulder_base_1.stl" scale="0.001 0.001 0.001"/>
+    </geometry>
+    <material name="silver"/>
+  </visual>
+  <collision>
+    <origin xyz="0.043637 -0.006593 -0.045671" rpy="0 0 0"/>
+    <geometry>
+      <mesh filename="$(find bartender_robot)/meshes/shoulder_base_1.stl" scale="0.001 0.001 0.001"/>
+    </geometry>
+  </collision>
+</link>
+<link name="shoulder_rotation_1">
+  <inertial>
+    <origin xyz="-0.05629632389205403 -1.4051646775835314e-07 0.05395678318861841" rpy="0 0 0"/>
+    <mass value="0.6894316761075354"/>
+    <inertia ixx="0.0017" iyy="0.000998" izz="0.00091" ixy="-0.0" iyz="0.0" ixz="-3e-05"/>
+  </inertial>
+  <visual>
+    <origin xyz="0.043637 -0.006593 -0.055671" rpy="0 0 0"/>
+    <geometry>
+      <mesh filename="$(find bartender_robot)/meshes/shoulder_rotation_1.stl" scale="0.001 0.001 0.001"/>
+    </geometry>
+    <material name="silver"/>
+  </visual>
+  <collision>
+    <origin xyz="0.043637 -0.006593 -0.055671" rpy="0 0 0"/>
+    <geometry>
+      <mesh filename="$(find bartender_robot)/meshes/shoulder_rotation_1.stl" scale="0.001 0.001 0.001"/>
+    </geometry>
+  </collision>
+</link>
+<link name="shoulder_motor_1">
+  <inertial>
+    <origin xyz="0.05614286278925305 -1.4051646683287816e-07 0.05301080568311395" rpy="0 0 0"/>
+    <mass value="0.6358704484213904"/>
+    <inertia ixx="0.001679" iyy="0.000976" izz="0.0009" ixy="-0.0" iyz="0.0" ixz="3.3e-05"/>
+  </inertial>
+  <visual>
+    <origin xyz="0.043637 -0.006593 -0.055671" rpy="0 0 0"/>
+    <geometry>
+      <mesh filename="$(find bartender_robot)/meshes/shoulder_motor_1.stl" scale="0.001 0.001 0.001"/>
+    </geometry>
+    <material name="silver"/>
+  </visual>
+  <collision>
+    <origin xyz="0.043637 -0.006593 -0.055671" rpy="0 0 0"/>
+    <geometry>
+      <mesh filename="$(find bartender_robot)/meshes/shoulder_motor_1.stl" scale="0.001 0.001 0.001"/>
+    </geometry>
+  </collision>
+</link>
+<link name="shoulder_motor_fix_1">
+  <inertial>
+    <origin xyz="-0.002000314055542886 -0.012250140516470387 -0.028250334635338367" rpy="0 0 0"/>
+    <mass value="0.009751151497809021"/>
+    <inertia ixx="8e-06" iyy="5e-06" izz="3e-06" ixy="-0.0" iyz="0.0" ixz="0.0"/>
+  </inertial>
+  <visual>
+    <origin xyz="0.007637 -0.018843 -0.151921" rpy="0 0 0"/>
+    <geometry>
+      <mesh filename="$(find bartender_robot)/meshes/shoulder_motor_fix_1.stl" scale="0.001 0.001 0.001"/>
+    </geometry>
+    <material name="silver"/>
+  </visual>
+  <collision>
+    <origin xyz="0.007637 -0.018843 -0.151921" rpy="0 0 0"/>
+    <geometry>
+      <mesh filename="$(find bartender_robot)/meshes/shoulder_motor_fix_1.stl" scale="0.001 0.001 0.001"/>
+    </geometry>
+  </collision>
+</link>
+<link name="XL_430_shoulder_1">
+  <inertial>
+    <origin xyz="0.014796642718762201 0.010999859483532937 -0.019917936953774626" rpy="0 0 0"/>
+    <mass value="0.34309933643690577"/>
+    <inertia ixx="8.2e-05" iyy="9.2e-05" izz="5.5e-05" ixy="-0.0" iyz="-0.0" ixz="-2e-06"/>
+  </inertial>
+  <visual>
+    <origin xyz="0.007637 0.004407 -0.143671" rpy="0 0 0"/>
+    <geometry>
+      <mesh filename="$(find bartender_robot)/meshes/XL_430_shoulder_1.stl" scale="0.001 0.001 0.001"/>
+    </geometry>
+    <material name="silver"/>
+  </visual>
+  <collision>
+    <origin xyz="0.007637 0.004407 -0.143671" rpy="0 0 0"/>
+    <geometry>
+      <mesh filename="$(find bartender_robot)/meshes/XL_430_shoulder_1.stl" scale="0.001 0.001 0.001"/>
+    </geometry>
+  </collision>
+</link>
+<link name="horn_shoulder_1">
+  <inertial>
+    <origin xyz="-0.0019564836971386317 -1.405164672153847e-07 -3.346353674993363e-07" rpy="0 0 0"/>
+    <mass value="0.009818206481012393"/>
+    <inertia ixx="0.0" iyy="0.0" izz="0.0" ixy="0.0" iyz="0.0" ixz="-0.0"/>
+  </inertial>
+  <visual>
+    <origin xyz="0.008937 -0.006593 -0.135671" rpy="0 0 0"/>
+    <geometry>
+      <mesh filename="$(find bartender_robot)/meshes/horn_shoulder_1.stl" scale="0.001 0.001 0.001"/>
+    </geometry>
+    <material name="silver"/>
+  </visual>
+  <collision>
+    <origin xyz="0.008937 -0.006593 -0.135671" rpy="0 0 0"/>
+    <geometry>
+      <mesh filename="$(find bartender_robot)/meshes/horn_shoulder_1.stl" scale="0.001 0.001 0.001"/>
+    </geometry>
+  </collision>
+</link>
+<link name="bearing_shoulder_1">
+  <inertial>
+    <origin xyz="0.004999685944448121 -1.405164666576711e-07 -3.34635320953236e-07" rpy="0 0 0"/>
+    <mass value="0.05186930462450643"/>
+    <inertia ixx="8e-06" iyy="4e-06" izz="4e-06" ixy="-0.0" iyz="0.0" ixz="0.0"/>
+  </inertial>
+  <visual>
+    <origin xyz="0.089637 -0.006593 -0.135671" rpy="0 0 0"/>
+    <geometry>
+      <mesh filename="$(find bartender_robot)/meshes/bearing_shoulder_1.stl" scale="0.001 0.001 0.001"/>
+    </geometry>
+    <material name="silver"/>
+  </visual>
+  <collision>
+    <origin xyz="0.089637 -0.006593 -0.135671" rpy="0 0 0"/>
+    <geometry>
+      <mesh filename="$(find bartender_robot)/meshes/bearing_shoulder_1.stl" scale="0.001 0.001 0.001"/>
+    </geometry>
+  </collision>
+</link>
+<link name="upper_arm_motor_1">
+  <inertial>
+    <origin xyz="-0.006254852404312311 -0.00447119946172419 -0.007927118189879956" rpy="0 0 0"/>
+    <mass value="0.0240331833914053"/>
+    <inertia ixx="1.5e-05" iyy="6e-06" izz="9e-06" ixy="-0.0" iyz="-0.0" ixz="-0.0"/>
+  </inertial>
+  <visual>
+    <origin xyz="0.012437 -0.006593 -0.135671" rpy="0 0 0"/>
+    <geometry>
+      <mesh filename="$(find bartender_robot)/meshes/upper_arm_motor_1.stl" scale="0.001 0.001 0.001"/>
+    </geometry>
+    <material name="silver"/>
+  </visual>
+  <collision>
+    <origin xyz="0.012437 -0.006593 -0.135671" rpy="0 0 0"/>
+    <geometry>
+      <mesh filename="$(find bartender_robot)/meshes/upper_arm_motor_1.stl" scale="0.001 0.001 0.001"/>
+    </geometry>
+  </collision>
+</link>
+<link name="XL_430_upper_1">
+  <inertial>
+    <origin xyz="0.007999685944452918 -0.006597097290772108 0.023332063046224677" rpy="0 0 0"/>
+    <mass value="0.34309933643690577"/>
+    <inertia ixx="9.2e-05" iyy="8.2e-05" izz="5.5e-05" ixy="0.0" iyz="2e-06" ixz="-0.0"/>
+  </inertial>
+  <visual>
+    <origin xyz="0.054437 0.004407 -0.100421" rpy="0 0 0"/>
+    <geometry>
+      <mesh filename="$(find bartender_robot)/meshes/XL_430_upper_1.stl" scale="0.001 0.001 0.001"/>
+    </geometry>
+    <material name="silver"/>
+  </visual>
+  <collision>
+    <origin xyz="0.054437 0.004407 -0.100421" rpy="0 0 0"/>
+    <geometry>
+      <mesh filename="$(find bartender_robot)/meshes/XL_430_upper_1.stl" scale="0.001 0.001 0.001"/>
+    </geometry>
+  </collision>
+</link>
+<link name="upper_arm_ceiling_1">
+  <inertial>
+    <origin xyz="-0.025125585660908684 0.013891988134250754 -0.005582870005646862" rpy="0 0 0"/>
+    <mass value="0.1422344344680632"/>
+    <inertia ixx="0.000112" iyy="0.0001" izz="0.000104" ixy="-0.0" iyz="1.2e-05" ixz="-0.0"/>
+  </inertial>
+  <visual>
+    <origin xyz="0.021437 0.011407 -0.137171" rpy="0 0 0"/>
+    <geometry>
+      <mesh filename="$(find bartender_robot)/meshes/upper_arm_ceiling_1.stl" scale="0.001 0.001 0.001"/>
+    </geometry>
+    <material name="silver"/>
+  </visual>
+  <collision>
+    <origin xyz="0.021437 0.011407 -0.137171" rpy="0 0 0"/>
+    <geometry>
+      <mesh filename="$(find bartender_robot)/meshes/upper_arm_ceiling_1.stl" scale="0.001 0.001 0.001"/>
+    </geometry>
+  </collision>
+</link>
+<link name="upper_arm_bottom_1">
+  <inertial>
+    <origin xyz="-0.019750314055547284 0.022437080248419432 -0.002471379083328562" rpy="0 0 0"/>
+    <mass value="0.024228655065312372"/>
+    <inertia ixx="1e-05" iyy="7e-06" izz="1.7e-05" ixy="0.0" iyz="0.0" ixz="-0.0"/>
+  </inertial>
+  <visual>
+    <origin xyz="0.026687 0.020907 -0.100421" rpy="0 0 0"/>
+    <geometry>
+      <mesh filename="$(find bartender_robot)/meshes/upper_arm_bottom_1.stl" scale="0.001 0.001 0.001"/>
+    </geometry>
+    <material name="silver"/>
+  </visual>
+  <collision>
+    <origin xyz="0.026687 0.020907 -0.100421" rpy="0 0 0"/>
+    <geometry>
+      <mesh filename="$(find bartender_robot)/meshes/upper_arm_bottom_1.stl" scale="0.001 0.001 0.001"/>
+    </geometry>
+  </collision>
+</link>
+<link name="upper_arm_rotation_1">
+  <inertial>
+    <origin xyz="-0.003232239536760731 0.03138877250113342 -0.011106481965935555" rpy="0 0 0"/>
+    <mass value="0.024156673189919837"/>
+    <inertia ixx="1.4e-05" iyy="6e-06" izz="9e-06" ixy="0.0" iyz="0.0" ixz="0.0"/>
+  </inertial>
+  <visual>
+    <origin xyz="0.071437 0.028407 -0.139171" rpy="0 0 0"/>
+    <geometry>
+      <mesh filename="$(find bartender_robot)/meshes/upper_arm_rotation_1.stl" scale="0.001 0.001 0.001"/>
+    </geometry>
+    <material name="silver"/>
+  </visual>
+  <collision>
+    <origin xyz="0.071437 0.028407 -0.139171" rpy="0 0 0"/>
+    <geometry>
+      <mesh filename="$(find bartender_robot)/meshes/upper_arm_rotation_1.stl" scale="0.001 0.001 0.001"/>
+    </geometry>
+  </collision>
+</link>
+<link name="horn_upper_1">
+  <inertial>
+    <origin xyz="-3.14055579167527e-07 0.001956029125128664 -3.346353356359355e-07" rpy="0 0 0"/>
+    <mass value="0.009818206481012393"/>
+    <inertia ixx="0.0" iyy="0.0" izz="0.0" ixy="0.0" iyz="0.0" ixz="-0.0"/>
+  </inertial>
+  <visual>
+    <origin xyz="0.046437 -0.005093 -0.135671" rpy="0 0 0"/>
+    <geometry>
+      <mesh filename="$(find bartender_robot)/meshes/horn_upper_1.stl" scale="0.001 0.001 0.001"/>
+    </geometry>
+    <material name="silver"/>
+  </visual>
+  <collision>
+    <origin xyz="0.046437 -0.005093 -0.135671" rpy="0 0 0"/>
+    <geometry>
+      <mesh filename="$(find bartender_robot)/meshes/horn_upper_1.stl" scale="0.001 0.001 0.001"/>
+    </geometry>
+  </collision>
+</link>
+<link name="lower_arm1_upper_1">
+  <inertial>
+    <origin xyz="-3.140555470890205e-07 0.03542416071948974 -3.3463535789590715e-07" rpy="0 0 0"/>
+    <mass value="0.09144869846484324"/>
+    <inertia ixx="5.8e-05" iyy="2.2e-05" izz="5.7e-05" ixy="-0.0" iyz="-0.0" ixz="0.0"/>
+  </inertial>
+  <visual>
+    <origin xyz="0.046437 -0.008593 -0.135671" rpy="0 0 0"/>
+    <geometry>
+      <mesh filename="$(find bartender_robot)/meshes/lower_arm1_upper_1.stl" scale="0.001 0.001 0.001"/>
+    </geometry>
+    <material name="silver"/>
+  </visual>
+  <collision>
+    <origin xyz="0.046437 -0.008593 -0.135671" rpy="0 0 0"/>
+    <geometry>
+      <mesh filename="$(find bartender_robot)/meshes/lower_arm1_upper_1.stl" scale="0.001 0.001 0.001"/>
+    </geometry>
+  </collision>
+</link>
+<link name="lower_arm1_lower2_1">
+  <inertial>
+    <origin xyz="0.01605879927304913 0.02717293837738126 -0.003950191764890698" rpy="0 0 0"/>
+    <mass value="0.07223595422977765"/>
+    <inertia ixx="4.1e-05" iyy="1.9e-05" izz="3.1e-05" ixy="-0.0" iyz="-0.0" ixz="0.0"/>
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