Commit message: update urdf

File: urdf_old/bartender_robot.xacro (robot description, xacro)
@@ -2,15 +2,16 @@
 <robot name="bartender_robot" xmlns:xacro="http://www.ros.org/wiki/xacro">
 <xacro:include filename="$(find bartender_robot)/urdf/materials.xacro" />
-<xacro:include filename="$(find bartender_robot)/urdf/bartender_robot.trans.xacro" />
+<xacro:include filename="$(find bartender_robot)/urdf/bartender_robot.trans" />
+<xacro:include filename="$(find bartender_robot)/urdf/bartender_robot.gazebo" />
 <link name="base_link">
   <inertial>
-    <origin xyz="-0.00040810804018468253 -3.552713678800501e-17 0.016706580181223032" rpy="0 0 0"/>
-    <mass value="6.935188631739772"/>
-    <inertia ixx="0.028142" iyy="0.028238" izz="0.054243" ixy="-0.0" iyz="-0.0" ixz="2.5e-05"/>
+    <origin xyz="-0.0005423501666184372 1.724031462449871e-05 0.021705683642274386" rpy="0 0 0"/>
+    <mass value="1.8079552496262552"/>
+    <inertia ixx="0.006993" iyy="0.007027" izz="0.013194" ixy="0.0" iyz="-0.0" ixz="3e-06"/>
   </inertial>
   <visual>
     <origin xyz="0 0 0" rpy="0 0 0"/>
     <geometry>
-  <mesh filename="package://bartender_robot/meshes/base_link.stl" scale="0.001 0.001 0.001"/>
+      <mesh filename="$(find bartender_robot)/meshes/base_link.stl" scale="0.001 0.001 0.001"/>
     </geometry>
     <material name="silver"/>
@@ -19,462 +20,1119 @@
     <origin xyz="0 0 0" rpy="0 0 0"/>
     <geometry>
-      <mesh filename="package://bartender_robot/meshes/base_link.stl" scale="0.001 0.001 0.001"/>
-    </geometry>
-  </collision>
-</link>
-<link name="motor_base_1">
-  <inertial>
-    <origin xyz="-0.011944616237443872 -1.1102230246251566e-17 0.016403799171755752" rpy="0 0 0"/>
-    <mass value="0.343534365338019"/>
-    <inertia ixx="5.5e-05" iyy="9.2e-05" izz="8.2e-05" ixy="-0.0" iyz="0.0" ixz="2e-06"/>
-  </inertial>
-  <visual>
-    <origin xyz="0.0 0.0 -0.015" rpy="0 0 0"/>
-    <geometry>
-  <mesh filename="package://bartender_robot/meshes/motor_base_1.stl" scale="0.001 0.001 0.001"/>
-    </geometry>
-    <material name="silver"/>
-  </visual>
-  <collision>
-    <origin xyz="0.0 0.0 -0.015" rpy="0 0 0"/>
-    <geometry>
-      <mesh filename="package://bartender_robot/meshes/motor_base_1.stl" scale="0.001 0.001 0.001"/>
-    </geometry>
-  </collision>
-</link>
-<link name="base_upperplate_1">
-  <inertial>
-    <origin xyz="-1.6172448750803435e-16 -3.676205142934621e-17 0.004999999999999949" rpy="0 0 0"/>
-    <mass value="1.9420933085410403"/>
-    <inertia ixx="0.007942" iyy="0.007942" izz="0.015852" ixy="-0.0" iyz="0.0" ixz="0.0"/>
-  </inertial>
-  <visual>
-    <origin xyz="0.0 0.0 -0.041" rpy="0 0 0"/>
-    <geometry>
-  <mesh filename="package://bartender_robot/meshes/base_upperplate_1.stl" scale="0.001 0.001 0.001"/>
-    </geometry>
-    <material name="silver"/>
-  </visual>
-  <collision>
-    <origin xyz="0.0 0.0 -0.041" rpy="0 0 0"/>
-    <geometry>
-      <mesh filename="package://bartender_robot/meshes/base_upperplate_1.stl" scale="0.001 0.001 0.001"/>
-    </geometry>
-  </collision>
-</link>
-<link name="motor_horn_base_1">
-  <inertial>
-    <origin xyz="3.138091383686708e-14 5.3428299048114016e-15 0.0019561696415957355" rpy="0 0 0"/>
+      <mesh filename="$(find bartender_robot)/meshes/base_link.stl" scale="0.001 0.001 0.001"/>
+    </geometry>
+  </collision>
+</link>
+<link name="horn_base_1">
+  <inertial>
+    <origin xyz="2.0834753222763892e-07 4.1573239855107635e-07 0.0019563297468164972" rpy="0 0 0"/>
+    <mass value="0.009818206481012393"/>
+    <inertia ixx="0.0" iyy="0.0" izz="0.0" ixy="-0.0" iyz="0.0" ixz="0.0"/>
+  </inertial>
+  <visual>
+    <origin xyz="-0.0 -0.0 -0.0475" rpy="0 0 0"/>
+    <geometry>
+      <mesh filename="$(find bartender_robot)/meshes/horn_base_1.stl" scale="0.001 0.001 0.001"/>
+    </geometry>
+    <material name="silver"/>
+  </visual>
+  <collision>
+    <origin xyz="-0.0 -0.0 -0.0475" rpy="0 0 0"/>
+    <geometry>
+      <mesh filename="$(find bartender_robot)/meshes/horn_base_1.stl" scale="0.001 0.001 0.001"/>
+    </geometry>
+  </collision>
+</link>
+<link name="shoulder_base_1">
+  <inertial>
+    <origin xyz="2.0834756958203033e-07 4.1573239849430243e-07 0.005013968553832557" rpy="0 0 0"/>
+    <mass value="0.38517204561220847"/>
+    <inertia ixx="0.000968" iyy="0.000958" izz="0.00192" ixy="0.0" iyz="0.0" ixz="-0.0"/>
+  </inertial>
+  <visual>
+    <origin xyz="-0.0 -0.0 -0.051" rpy="0 0 0"/>
+    <geometry>
+      <mesh filename="$(find bartender_robot)/meshes/shoulder_base_1.stl" scale="0.001 0.001 0.001"/>
+    </geometry>
+    <material name="silver"/>
+  </visual>
+  <collision>
+    <origin xyz="-0.0 -0.0 -0.051" rpy="0 0 0"/>
+    <geometry>
+      <mesh filename="$(find bartender_robot)/meshes/shoulder_base_1.stl" scale="0.001 0.001 0.001"/>
+    </geometry>
+  </collision>
+</link>
+<link name="shoulder_rotation_1">
+  <inertial>
+    <origin xyz="-0.05629580148894291 4.1573239737157185e-07 0.05395727792919584" rpy="0 0 0"/>
+    <mass value="0.6894316761075353"/>
+    <inertia ixx="0.0017" iyy="0.000998" izz="0.00091" ixy="-0.0" iyz="0.0" ixz="-3e-05"/>
+  </inertial>
+  <visual>
+    <origin xyz="-0.0 -0.0 -0.061" rpy="0 0 0"/>
+    <geometry>
+      <mesh filename="$(find bartender_robot)/meshes/shoulder_rotation_1.stl" scale="0.001 0.001 0.001"/>
+    </geometry>
+    <material name="silver"/>
+  </visual>
+  <collision>
+    <origin xyz="-0.0 -0.0 -0.061" rpy="0 0 0"/>
+    <geometry>
+      <mesh filename="$(find bartender_robot)/meshes/shoulder_rotation_1.stl" scale="0.001 0.001 0.001"/>
+    </geometry>
+  </collision>
+</link>
+<link name="shoulder_motor_1">
+  <inertial>
+    <origin xyz="0.056143385192364115 4.1573239833766036e-07 0.0530113004236914" rpy="0 0 0"/>
+    <mass value="0.6358704484213904"/>
+    <inertia ixx="0.001679" iyy="0.000976" izz="0.0009" ixy="-0.0" iyz="0.0" ixz="3.3e-05"/>
+  </inertial>
+  <visual>
+    <origin xyz="-0.0 -0.0 -0.061" rpy="0 0 0"/>
+    <geometry>
+      <mesh filename="$(find bartender_robot)/meshes/shoulder_motor_1.stl" scale="0.001 0.001 0.001"/>
+    </geometry>
+    <material name="silver"/>
+  </visual>
+  <collision>
+    <origin xyz="-0.0 -0.0 -0.061" rpy="0 0 0"/>
+    <geometry>
+      <mesh filename="$(find bartender_robot)/meshes/shoulder_motor_1.stl" scale="0.001 0.001 0.001"/>
+    </geometry>
+  </collision>
+</link>
+<link name="shoulder_motor_fix_1">
+  <inertial>
+    <origin xyz="-0.0019997916524318246 -0.01224958426760502 -0.028249839894760903" rpy="0 0 0"/>
+    <mass value="0.009751151497809021"/>
+    <inertia ixx="8e-06" iyy="5e-06" izz="3e-06" ixy="-0.0" iyz="0.0" ixz="-0.0"/>
+  </inertial>
+  <visual>
+    <origin xyz="-0.036 -0.01225 -0.15725" rpy="0 0 0"/>
+    <geometry>
+      <mesh filename="$(find bartender_robot)/meshes/shoulder_motor_fix_1.stl" scale="0.001 0.001 0.001"/>
+    </geometry>
+    <material name="silver"/>
+  </visual>
+  <collision>
+    <origin xyz="-0.036 -0.01225 -0.15725" rpy="0 0 0"/>
+    <geometry>
+      <mesh filename="$(find bartender_robot)/meshes/shoulder_motor_fix_1.stl" scale="0.001 0.001 0.001"/>
+    </geometry>
+  </collision>
+</link>
+<link name="XL_430_shoulder_1">
+  <inertial>
+    <origin xyz="0.014797165121873311 0.011000415732398234 -0.019917442213197245" rpy="0 0 0"/>
+    <mass value="0.34309933643690577"/>
+    <inertia ixx="8.2e-05" iyy="9.2e-05" izz="5.5e-05" ixy="-0.0" iyz="0.0" ixz="-2e-06"/>
+  </inertial>
+  <visual>
+    <origin xyz="-0.036 0.011 -0.149" rpy="0 0 0"/>
+    <geometry>
+      <mesh filename="$(find bartender_robot)/meshes/XL_430_shoulder_1.stl" scale="0.001 0.001 0.001"/>
+    </geometry>
+    <material name="silver"/>
+  </visual>
+  <collision>
+    <origin xyz="-0.036 0.011 -0.149" rpy="0 0 0"/>
+    <geometry>
+      <mesh filename="$(find bartender_robot)/meshes/XL_430_shoulder_1.stl" scale="0.001 0.001 0.001"/>
+    </geometry>
+  </collision>
+</link>
+<link name="horn_shoulder_1">
+  <inertial>
+    <origin xyz="-0.0019559612940275445 4.15732398126384e-07 1.6010520997866706e-07" rpy="0 0 0"/>
+    <mass value="0.009818206481012393"/>
+    <inertia ixx="0.0" iyy="0.0" izz="0.0" ixy="0.0" iyz="0.0" ixz="-0.0"/>
+  </inertial>
+  <visual>
+    <origin xyz="-0.0347 -0.0 -0.141" rpy="0 0 0"/>
+    <geometry>
+      <mesh filename="$(find bartender_robot)/meshes/horn_shoulder_1.stl" scale="0.001 0.001 0.001"/>
+    </geometry>
+    <material name="silver"/>
+  </visual>
+  <collision>
+    <origin xyz="-0.0347 -0.0 -0.141" rpy="0 0 0"/>
+    <geometry>
+      <mesh filename="$(find bartender_robot)/meshes/horn_shoulder_1.stl" scale="0.001 0.001 0.001"/>
+    </geometry>
+  </collision>
+</link>
+<link name="bearing_shoulder_1">
+  <inertial>
+    <origin xyz="0.0050002083475592166 4.157323989105617e-07 1.6010525652476737e-07" rpy="0 0 0"/>
+    <mass value="0.05186930462450643"/>
+    <inertia ixx="8e-06" iyy="4e-06" izz="4e-06" ixy="-0.0" iyz="0.0" ixz="0.0"/>
+  </inertial>
+  <visual>
+    <origin xyz="0.046 -0.0 -0.141" rpy="0 0 0"/>
+    <geometry>
+      <mesh filename="$(find bartender_robot)/meshes/bearing_shoulder_1.stl" scale="0.001 0.001 0.001"/>
+    </geometry>
+    <material name="silver"/>
+  </visual>
+  <collision>
+    <origin xyz="0.046 -0.0 -0.141" rpy="0 0 0"/>
+    <geometry>
+      <mesh filename="$(find bartender_robot)/meshes/bearing_shoulder_1.stl" scale="0.001 0.001 0.001"/>
+    </geometry>
+  </collision>
+</link>
+<link name="upper_arm_motor_1">
+  <inertial>
+    <origin xyz="-0.006254330001201239 -0.00447064321285894 -0.007926623449302533" rpy="0 0 0"/>
+    <mass value="0.0240331833914053"/>
+    <inertia ixx="1.5e-05" iyy="6e-06" izz="9e-06" ixy="-0.0" iyz="-0.0" ixz="-0.0"/>
+  </inertial>
+  <visual>
+    <origin xyz="-0.0312 -0.0 -0.141" rpy="0 0 0"/>
+    <geometry>
+      <mesh filename="$(find bartender_robot)/meshes/upper_arm_motor_1.stl" scale="0.001 0.001 0.001"/>
+    </geometry>
+    <material name="silver"/>
+  </visual>
+  <collision>
+    <origin xyz="-0.0312 -0.0 -0.141" rpy="0 0 0"/>
+    <geometry>
+      <mesh filename="$(find bartender_robot)/meshes/upper_arm_motor_1.stl" scale="0.001 0.001 0.001"/>
+    </geometry>
+  </collision>
+</link>
+<link name="XL_430_upper_1">
+  <inertial>
+    <origin xyz="0.008000208347564024 -0.006596541041906951 0.023332557786802058" rpy="0 0 0"/>
+    <mass value="0.34309933643690577"/>
+    <inertia ixx="9.2e-05" iyy="8.2e-05" izz="5.5e-05" ixy="0.0" iyz="2e-06" ixz="-0.0"/>
+  </inertial>
+  <visual>
+    <origin xyz="0.0108 0.011 -0.10575" rpy="0 0 0"/>
+    <geometry>
+      <mesh filename="$(find bartender_robot)/meshes/XL_430_upper_1.stl" scale="0.001 0.001 0.001"/>
+    </geometry>
+    <material name="silver"/>
+  </visual>
+  <collision>
+    <origin xyz="0.0108 0.011 -0.10575" rpy="0 0 0"/>
+    <geometry>
+      <mesh filename="$(find bartender_robot)/meshes/XL_430_upper_1.stl" scale="0.001 0.001 0.001"/>
+    </geometry>
+  </collision>
+</link>
+<link name="upper_arm_ceiling_1">
+  <inertial>
+    <origin xyz="-0.025125063257797613 0.013892544383116098 -0.005582375265069439" rpy="0 0 0"/>
+    <mass value="0.1422344344680632"/>
+    <inertia ixx="0.000112" iyy="0.0001" izz="0.000104" ixy="-0.0" iyz="1.2e-05" ixz="-0.0"/>
+  </inertial>
+  <visual>
+    <origin xyz="-0.0222 0.018 -0.1425" rpy="0 0 0"/>
+    <geometry>
+      <mesh filename="$(find bartender_robot)/meshes/upper_arm_ceiling_1.stl" scale="0.001 0.001 0.001"/>
+    </geometry>
+    <material name="silver"/>
+  </visual>
+  <collision>
+    <origin xyz="-0.0222 0.018 -0.1425" rpy="0 0 0"/>
+    <geometry>
+      <mesh filename="$(find bartender_robot)/meshes/upper_arm_ceiling_1.stl" scale="0.001 0.001 0.001"/>
+    </geometry>
+  </collision>
+</link>
+<link name="upper_arm_bottom_1">
+  <inertial>
+    <origin xyz="-0.019749791652436222 0.022437636497284773 -0.0024708843427511257" rpy="0 0 0"/>
+    <mass value="0.024228655065312372"/>
+    <inertia ixx="1e-05" iyy="7e-06" izz="1.7e-05" ixy="-0.0" iyz="0.0" ixz="-0.0"/>
+  </inertial>
+  <visual>
+    <origin xyz="-0.01695 0.0275 -0.10575" rpy="0 0 0"/>
+    <geometry>
+      <mesh filename="$(find bartender_robot)/meshes/upper_arm_bottom_1.stl" scale="0.001 0.001 0.001"/>
+    </geometry>
+    <material name="silver"/>
+  </visual>
+  <collision>
+    <origin xyz="-0.01695 0.0275 -0.10575" rpy="0 0 0"/>
+    <geometry>
+      <mesh filename="$(find bartender_robot)/meshes/upper_arm_bottom_1.stl" scale="0.001 0.001 0.001"/>
+    </geometry>
+  </collision>
+</link>
+<link name="upper_arm_rotation_1">
+  <inertial>
+    <origin xyz="-0.0032317171336496524 0.03138932874999876 -0.011105987225358105" rpy="0 0 0"/>
+    <mass value="0.024156673189919837"/>
+    <inertia ixx="1.4e-05" iyy="6e-06" izz="9e-06" ixy="0.0" iyz="0.0" ixz="0.0"/>
+  </inertial>
+  <visual>
+    <origin xyz="0.0278 0.035 -0.1445" rpy="0 0 0"/>
+    <geometry>
+      <mesh filename="$(find bartender_robot)/meshes/upper_arm_rotation_1.stl" scale="0.001 0.001 0.001"/>
+    </geometry>
+    <material name="silver"/>
+  </visual>
+  <collision>
+    <origin xyz="0.0278 0.035 -0.1445" rpy="0 0 0"/>
+    <geometry>
+      <mesh filename="$(find bartender_robot)/meshes/upper_arm_rotation_1.stl" scale="0.001 0.001 0.001"/>
+    </geometry>
+  </collision>
+</link>
+<link name="horn_upper_1">
+  <inertial>
+    <origin xyz="2.0834753190063227e-07 0.001956585373994231 1.601052418143123e-07" rpy="0 0 0"/>
+    <mass value="0.009818206481012393"/>
+    <inertia ixx="0.0" iyy="0.0" izz="0.0" ixy="0.0" iyz="0.0" ixz="-0.0"/>
+  </inertial>
+  <visual>
+    <origin xyz="0.0028 0.0015 -0.141" rpy="0 0 0"/>
+    <geometry>
+      <mesh filename="$(find bartender_robot)/meshes/horn_upper_1.stl" scale="0.001 0.001 0.001"/>
+    </geometry>
+    <material name="silver"/>
+  </visual>
+  <collision>
+    <origin xyz="0.0028 0.0015 -0.141" rpy="0 0 0"/>
+    <geometry>
+      <mesh filename="$(find bartender_robot)/meshes/horn_upper_1.stl" scale="0.001 0.001 0.001"/>
+    </geometry>
+  </collision>
+</link>
+<link name="lower_arm1_upper_1">
+  <inertial>
+    <origin xyz="2.0834756397610302e-07 0.03542471696835489 1.6010521958209623e-07" rpy="0 0 0"/>
+    <mass value="0.09144869846484324"/>
+    <inertia ixx="5.8e-05" iyy="2.2e-05" izz="5.7e-05" ixy="-0.0" iyz="-0.0" ixz="0.0"/>
+  </inertial>
+  <visual>
+    <origin xyz="0.0028 -0.002 -0.141" rpy="0 0 0"/>
+    <geometry>
+      <mesh filename="$(find bartender_robot)/meshes/lower_arm1_upper_1.stl" scale="0.001 0.001 0.001"/>
+    </geometry>
+    <material name="silver"/>
+  </visual>
+  <collision>
+    <origin xyz="0.0028 -0.002 -0.141" rpy="0 0 0"/>
+    <geometry>
+      <mesh filename="$(find bartender_robot)/meshes/lower_arm1_upper_1.stl" scale="0.001 0.001 0.001"/>
+    </geometry>
+  </collision>
+</link>
+<link name="lower_arm1_lower2_1">
+  <inertial>
+    <origin xyz="0.016058321676160184 0.02717349462624645 -0.003950697024313138" rpy="0 0 0"/>
+    <mass value="0.07223595422977765"/>
+    <inertia ixx="4.1e-05" iyy="1.9e-05" izz="3.1e-05" ixy="-0.0" iyz="-0.0" ixz="0.0"/>
+  </inertial>
+  <visual>
+    <origin xyz="0.018812 -0.082 -0.144951" rpy="0 0 0"/>
+    <geometry>
+      <mesh filename="$(find bartender_robot)/meshes/lower_arm1_lower2_1.stl" scale="0.001 0.001 0.001"/>
+    </geometry>
+    <material name="silver"/>
+  </visual>
+  <collision>
+    <origin xyz="0.018812 -0.082 -0.144951" rpy="0 0 0"/>
+    <geometry>
+      <mesh filename="$(find bartender_robot)/meshes/lower_arm1_lower2_1.stl" scale="0.001 0.001 0.001"/>
+    </geometry>
+  </collision>
+</link>
+<link name="XL_430_lower1_1">
+  <inertial>
+    <origin xyz="0.0065529356146676095 -0.007917186586020197 0.014270785373014377" rpy="0 0 0"/>
+    <mass value="0.34309933643690577"/>
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